Commit message: URDF of the robot bridge updated with the Hokuyo support

File: model/gazebo/Bridge.urdf.xacro (robot description, xacro)
@@ -13,5 +13,5 @@
         <inertial>
           <origin
-            xyz="0.0636736810906936 0.143842323651452 0.00299999999999712"
+            xyz="0.0636736810906936 0.143842323651452 0.00299999999999717"
             rpy="0 0 0" />
           <mass
@@ -19,8 +19,8 @@
           <inertia
             ixx="0.00152014852697095"
-            ixy="1.76846639004149E-05"
-            ixz="-3.1539863417057E-18"
+            ixy="1.76846639004148E-05"
+            ixz="-3.15136020868249E-18"
             iyy="0.000286140203372851"
-            iyz="-2.34660601836366E-17"
+            iyz="-2.34411025118014E-17"
             izz="0.00180507409034381" />
         </inertial>
@@ -52,14 +52,14 @@
         <inertial>
           <origin
-            xyz="0.0540874050204184 0.178160355074789 0.00302783690149616"
+            xyz="-0.0976625949795816 0.178160355074788 0.00302783690149633"
             rpy="0 0 0" />
           <mass
             value="0.192741498658911" />
           <inertia
-            ixx="0.00247517327495455"
-            ixy="-0.000307984645851293"
-            ixz="1.41948006226161E-08"
-            iyy="0.000287632943939697"
-            iyz="-1.60207534296156E-07"
+            ixx="0.00247517327495454"
+            ixy="-0.000307984645851296"
+            ixz="1.41948006227713E-08"
+            iyy="0.000287632943939698"
+            iyz="-1.60207534296806E-07"
             izz="0.0027616214535378" />
         </inertial>
@@ -90,6 +90,6 @@
       <joint name="robot_bridge_left_joint" type="fixed">
         <origin
-          xyz="0.15 0.286000000000024 0"
-          rpy="1.57079632679491 -1.62922021519875E-15 3.14159265358979" />
+          xyz="-0.0017499999999999 0.286000000000004 0"
+          rpy="1.57079632679491 -4.98180625530473E-16 3.14159265358979" />
         <parent
           link="robot_bridge" />
@@ -97,10 +97,10 @@
           link="robot_bridge_left" />
         <axis
-          xyz="0 0 0" />
+          xyz="1 0 0" />
       </joint>
       <link name="robot_bridge_right">
         <inertial>
           <origin
-            xyz="0.0540874050204184 0.178160355074789 0.00302783690149645"
+            xyz="0.0540874050204185 0.178160355074789 0.00302783690149646"
             rpy="0 0 0" />
           <mass
@@ -109,5 +109,5 @@
             ixx="0.00247517327495456"
             ixy="-0.000307984645851296"
-            ixz="1.41948006226808E-08"
+            ixz="1.41948006224639E-08"
             iyy="0.000287632943939699"
             iyz="-1.6020753429316E-07"
@@ -151,15 +151,14 @@
       <link name="robot_bridge_top">
         <inertial>
-          <origin
-            xyz="0.146 0.0250000000000003 0.003000000000001"
-            rpy="0 0 0" />
+          <origin xyz="0.146 0.0250000000000003 0.003000000000001" rpy="0 0 0" />
+<!--          <origin xyz="0.14 0.0979999999999973 0.397000000000002" rpy="0 0 0" />-->
           <mass
             value="0.0861599999999999" />
           <inertia
             ixx="1.846048E-05"
-            ixy="1.09436656785256E-18"
-            ixz="4.63938687723111E-18"
+            ixy="1.09563711727344E-18"
+            ixz="4.63866741667959E-18"
             iyy="0.0005932348"
-            iyz="-1.8841390206596E-19"
+            iyz="-1.88171846788368E-19"
             izz="0.00061117832" />
         </inertial>
@@ -189,7 +188,6 @@
       </gazebo>
       <joint name="robot_bridge_top_joint" type="fixed">
-        <origin
-          xyz="0.100000000000004 0.291999999999986 0.394000000000001"
-          rpy="0 0 -1.5707963267949" />
+<!--        <origin xyz="0.0270000000000069 0.286000000000004 0" rpy="0 0 -1.5707963267949" />-->
+        <origin xyz="0.100000000000004 0.291999999999986 0.394000000000001" rpy="0 0 -1.5707963267949" />
         <parent
           link="robot_bridge" />
@@ -197,106 +195,170 @@
           link="robot_bridge_top" />
         <axis
+          xyz="0 -1 0" />
+      </joint>
+      <link name="robot_bridge_box">
+        <inertial>
+          <origin
+            xyz="0.0508000000000002 0.139700000000001 0.0888999999999976"
+            rpy="0 0 0" />
+          <mass
+            value="5.047215712" />
+          <inertia
+            ixx="0.0461303739240139"
+            ixy="-1.0842021724855E-17"
+            ixz="1.74874855526867E-17"
+            iyy="0.0176380841474171"
+            iyz="-3.00743891293254E-16"
+            izz="0.0371756542799406" />
+        </inertial>
+        <visual>
+          <origin
+            xyz="0 0 0"
+            rpy="0 0 0" />
+          <geometry>
+            <mesh
+              filename="package://hratc2017_robot/model/gazebo/meshes/Box.STL" />
+          </geometry>
+          <material name="color_bridge1" />
+        </visual>
+        <collision>
+          <origin
+            xyz="0 0 0"
+            rpy="0 0 0" />
+          <geometry>
+            <mesh
+              filename="package://hratc2017_robot/model/gazebo/meshes/Box.STL" />
+          </geometry>
+        </collision>
+      </link>
+      <gazebo reference="robot_bridge_box">
+        <material>Gazebo/FlatBlack</material>
+        <turnGravityOff>false</turnGravityOff>
+      </gazebo>
+      <joint name="robot_bridge_box_joint" type="fixed">
+        <origin
+          xyz="0.0314250374432209 0.00600000000000061 0.0426820783873315"
+          rpy="0 0 -2.77555756156289E-17" />
+        <parent
+          link="robot_bridge" />
+        <child
+          link="robot_bridge_box" />
+        <axis
           xyz="0 0 0" />
       </joint>
-      <link name="robot_bridge_box">
-        <inertial>
-          <origin
-            xyz="0.0508000000000001 0.139700000000001 0.0888999999999978"
-            rpy="0 0 0" />
-          <mass
-            value="5.047215712" />
-          <inertia
-            ixx="0.0461303739240139"
-            ixy="-9.10729824887824E-18"
-            ixz="1.55504347364085E-17"
-            iyy="0.0176380841474171"
-            iyz="-2.98372626157703E-16"
-            izz="0.0371756542799406" />
-        </inertial>
-        <visual>
-          <origin
-            xyz="0 0 0"
-            rpy="0 0 0" />
-          <geometry>
-            <mesh
-              filename="package://hratc2017_robot/model/gazebo/meshes/Box.STL" />
-          </geometry>
-          <material name="color_bridge1" />
-        </visual>
-        <collision>
-          <origin
-            xyz="0 0 0"
-            rpy="0 0 0" />
-          <geometry>
-            <mesh
-              filename="package://hratc2017_robot/model/gazebo/meshes/Box.STL" />
-          </geometry>
-        </collision>
-      </link>
-      <gazebo reference="robot_bridge_box">
-        <material>Gazebo/FlatBlack</material>
-        <turnGravityOff>false</turnGravityOff>
-      </gazebo>
-      <joint name="robot_bridge_box_joint" type="fixed">
-        <origin
-          xyz="0.0314250374432224 0.00600000000000064 0.0426820783873312"
-          rpy="0 0 -2.77555756156289E-17" />
-        <parent
-          link="robot_bridge" />
-        <child
-          link="robot_bridge_box" />
+      <link
+        name="Hokuyo_support">
+        <inertial>
+          <origin
+            xyz="0.025 0.0143387096774193 -0.01"
+            rpy="0 0 0" />
+          <mass
+            value="0.031" />
+          <inertia
+            ixx="7.79011021505377E-06"
+            ixy="-3.3230248811664E-21"
+            ixz="3.17637355220355E-21"
+            iyy="1.24916666666667E-05"
+            iyz="2.01326094458915E-21"
+            izz="8.21511021505378E-06" />
+        </inertial>
+        <visual>
+          <origin
+            xyz="0 0 0"
+            rpy="0 0 0" />
+          <geometry>
+            <mesh
+              filename="package://hratc2017_robot/model/gazebo/meshes/Hokuyo_support.STL" />
+          </geometry>
+          <material
+            name="">
+            <color
+              rgba="0.792156862745098 0.819607843137255 0.933333333333333 1" />
+          </material>
+        </visual>
+        <collision>
+          <origin
+            xyz="0 0 0"
+            rpy="0 0 0" />
+          <geometry>
+            <mesh
+              filename="package://hratc2017_robot/model/gazebo/meshes/Hokuyo_support.STL" />
+          </geometry>
+        </collision>
+      </link>
+      <gazebo reference="Hokuyo_support">
+        <material>Gazebo/FlatBlack</material>
+        <turnGravityOff>false</turnGravityOff>
+      </gazebo>
+      <joint
+        name="Hokuyo_support_joint"
+        type="fixed">
+        <origin
+          xyz="0.155425037443221 0.138000000000004 0.245482078387329"
+          rpy="-1.57079632679488 -9.10853057488072E-16 -3.14159265358979" />
+        <parent
+          link="robot_bridge" />
+        <child
+          link="Hokuyo_support" />
         <axis
           xyz="0 0 0" />
       </joint>
-<!--      <link name="Laser_support">-->
-<!--        <inertial>-->
-<!--          <origin-->
-<!--            xyz="0.0450000000000004 0.0265300391501749 -0.047447780251052"-->
-<!--            rpy="0 0 0" />-->
-<!--          <mass-->
-<!--            value="0.077668648558694" />-->
-<!--          <inertia-->
-<!--            ixx="0.000240204828475503"-->
-<!--            ixy="-1.21972744404628E-19"-->
-<!--            ixz="-1.51216556908574E-18"-->
-<!--            iyy="0.000248773184670883"-->
-<!--            iyz="1.39921616907987E-05"-->
-<!--            izz="0.000101877527595527" />-->
-<!--        </inertial>-->
-<!--        <visual>-->
-<!--          <origin-->
-<!--            xyz="0 0 0"-->
-<!--            rpy="0 0 0" />-->
-<!--          <geometry>-->
-<!--            <mesh-->
-<!--              filename="package://hratc2017_robot/model/gazebo/meshes/Laser_support.STL" />-->
-<!--          </geometry>-->
-<!--          <material name="color_bridge1" />-->
-<!--        </visual>-->
-<!--        <collision>-->
-<!--          <origin-->
-<!--            xyz="0 0 0"-->
-<!--            rpy="0 0 0" />-->
-<!--          <geometry>-->
-<!--            <mesh-->
-<!--              filename="package://hratc2017_robot/model/gazebo/meshes/Laser_support.STL" />-->
-<!--          </geometry>-->
-<!--        </collision>-->
-<!--      </link>-->
-<!--      <gazebo reference="Laser_support">-->
-<!--        <material>Gazebo/FlatBlack</material>-->
-<!--        <turnGravityOff>false</turnGravityOff>-->
-<!--      </gazebo>-->
-<!--      <joint name="Laser_support_joint" type="fixed">-->
-<!--        <origin-->
-<!--          xyz="0.0820581161712757 0.113821575351547 0.405000000000003"-->
-<!--          rpy="-3.14159265358978 0 1.52865875946308" />-->
-<!--        <parent-->
-<!--          link="robot_bridge" />-->
-<!--        <child-->
-<!--          link="Laser_support" />-->
-<!--        <axis-->
-<!--          xyz="0 0 0" />-->
-<!--      </joint>-->
+      <link
+        name="Hokuyo_joint">
+        <inertial>
+          <origin
+            xyz="0.0100000000000001 0.0305650668622638 0.01"
+            rpy="0 0 0" />
+          <mass
+            value="0.0278046900494077" />
+          <inertia
+            ixx="8.27124323386541E-06"
+            ixy="8.470329472543E-22"
+            ixz="1.198203476133E-21"
+            iyy="6.20545766519684E-06"
+            iyz="-2.83844472876361E-21"
+            izz="8.2480548957684E-06" />
+        </inertial>
+        <visual>
+          <origin
+            xyz="0 0 0"
+            rpy="0 0 0" />
+          <geometry>
+            <mesh
+              filename="package://hratc2017_robot/model/gazebo/meshes/Hokuyo_joint.STL" />
+          </geometry>
+          <material
+            name="">
+            <color
+              rgba="0.792156862745098 0.819607843137255 0.933333333333333 1" />
+          </material>
+        </visual>
+        <collision>
+          <origin
+            xyz="0 0 0"
+            rpy="0 0 0" />
+          <geometry>
+            <mesh
+              filename="package://hratc2017_robot/model/gazebo/meshes/Hokuyo_joint.STL" />
+          </geometry>
+        </collision>
+      </link>
+      <gazebo reference="Hokuyo_joint">
+        <material>Gazebo/FlatBlack</material>
+        <turnGravityOff>false</turnGravityOff>
+      </gazebo>
+      <joint
+        name="Hokuyo_joint_joint"
+        type="fixed">
+        <origin
+          xyz="0.0238411453116162 0.0110630275987395 -0.02"
+          rpy="3.5586180135377E-16 -9.75292147983034E-16 2.53072741539178" />
+        <parent
+          link="Hokuyo_support" />
+        <child
+          link="Hokuyo_joint" />
+        <axis
+          xyz="0 0 0" />
+      </joint>
     </xacro:macro>
 </robot>
