Commit message: changed definitions for the pioneer3at urdf

File: description/urdf/urdf/mti.urdf.xacro (robot description, xacro)
@@ -60,5 +60,5 @@
             <plugin name="gazebo_ros_imu" filename="libgazebo_ros_imu.so">
                 <alwaysOn>true</alwaysOn>
-                <bodyName>base_link</bodyName>
+                <bodyName>base_footprint</bodyName>
                 <topicName>/imu/data</topicName>
                 <serviceName>imu_service</serviceName>

File: description/urdf/urdf/pioneer3at.urdf.xacro (robot description, xacro)
@@ -13,4 +13,29 @@
 <xacro:include filename="$(find metal_detector_msgs)/model/gazebo/metal_detector.urdf.xacro" />
 <xacro:include filename="$(find hratc2017_robot)/model/gazebo/Bridge.urdf.xacro" />
+    <!-- BASE-FOOTPRINT -->
+    <!-- base_footprint is a fictitious link(frame) that is on the ground right below base_link origin, navigation stack depends on this frame -->
+    <link name="base_footprint">
+        <!--<inertial>
+            <mass value="0.0001" />
+            <origin xyz="0 0 0" />
+            <inertia ixx="0.0001" ixy="0.0" ixz="0.0"
+                iyy="0.0001" iyz="0.0"
+                izz="0.0001" />
+	      </inertial>-->
+        <visual>
+            <origin xyz="0 0 0" rpy="0 0 0" />
+            <geometry>
+                <box size="0.001 0.001 0.001" />
+            </geometry>
+        </visual>
+    </link>
+    <gazebo reference="base_footprint">
+        <turnGravityOff>false</turnGravityOff>
+    </gazebo>
+    <joint name="base_footprint_joint" type="fixed">
+		<origin xyz="0 0 0" rpy="0 0 0" />
+        <parent link="base_footprint"/>
+        <child link="base_link" />
+    </joint>
 <!-- Chassis -->
     <link name="base_link">
